Commit message: urdf

File: legged_gym/resources/robots/panda7/urdf/panda7_nleg_arm_1008.urdf (robot description, URDF)
Before this commit: robot panda7, 26 links, 25 joints
Links:
- added link imu, mass 0.1; visual box size=0.015 0.015 0.004
- link FL_FOOT: mass 0.01 -> 0.12
- link FR_FOOT: mass 0.01 -> 0.12
- link RL_FOOT: mass 0.01 -> 0.12
- link RR_FOOT: mass 0.01 -> 0.12
- link arm_link0: geometry visual mesh filename=../meshes/link0.dae
- link arm_link1: geometry visual mesh filename=../meshes/link1.dae
- link arm_link2: geometry visual mesh filename=../meshes/link2.dae
- link arm_link3: geometry visual mesh filename=../meshes/link3.dae
- link arm_link4: mass 0.0428548065855341 -> 0.042855; geometry visual mesh filename=../meshes/link4.dae
- link arm_link5: geometry visual mesh filename=../meshes/link5.dae
- link arm_link6: geometry visual mesh filename=../meshes/link6.dae
- link gripper1: geometry visual mesh filename=../meshes/gripper1.dae
- link gripper2: geometry visual mesh filename=../meshes/gripper2.dae
Joints:
- added joint imu_joint: type fixed, parent base, child imu, origin xyz=0. 0. 0. rpy=0. 0. 0.
- joint arm_joint4: origin xyz=0.251713743388397 -0.0670979052394916 0 rpy=0 0 0 -> xyz=0.245 -0.056 -0.000475 rpy=0 0 0
- joint arm_joint5: origin xyz=0.0600362566116027 -0.0729020947605091 -0.0504267019672398 rpy=1.5707963267949 1.5707963267949 0 -> xyz=0.06675 -0.084 -0.000275 rpy=1.5708 1.5708 0

File: legged_gym/resources/robots/panda7_fixed_gripper/urdf/panda7_nleg_arm_1008.urdf (robot description, URDF)
Before this commit: robot robot, 27 links, 26 joints
Links:
- link FL_FOOT: mass 0.0001 -> 0.12
- link FR_FOOT: mass 0.0001 -> 0.12
- link RL_FOOT: mass 0.0001 -> 0.12
- link RR_FOOT: mass 0.0001 -> 0.12
- link imu: mass 0.01 -> 0.1
Joints:
- joint arm_joint7: type prismatic -> fixed
- joint arm_joint8: type prismatic -> fixed
